Commit message: Signed-off-by: Or Tslil <ortslil64@gmail.com>

File: urdf/KoBot_ai.urdf.xacro (robot description, xacro)
@@ -15,13 +15,13 @@
   </inertial>
   <visual>
-    <origin xyz="0 0 0.17"/>
-    <geometry>
-      <box size="0.8 0.545 0.17" />
+    <origin xyz="0 0 0.125"/>
+    <geometry>
+      <box size="0.8 0.545 0.1" />
     </geometry>
   </visual>
   <collision>
-    <origin xyz="0 0 0.17"/>
-    <geometry>
-      <box size="0.8 0.545 0.17" />
+    <origin xyz="0 0 0.125"/>
+    <geometry>
+      <box size="0.8 0.545 0.1" />
     </geometry>
   </collision>
@@ -39,5 +39,5 @@
     <origin rpy="1.5707963267948966 0 0" xyz="0 0 0"/>
     <geometry>
-      <cylinder length="0.05" radius="0.12"/>
+      <cylinder length="0.05" radius="0.1"/>
     </geometry>
   </visual>
@@ -45,5 +45,5 @@
     <origin rpy="1.5707963267948966 0 0" xyz="0 0 0"/>
     <geometry>
-      <cylinder length="0.05" radius="0.12"/>
+      <cylinder length="0.05" radius="0.1"/>
     </geometry>
   </collision>
@@ -77,5 +77,5 @@
     <origin rpy="1.5707963267948966 0 0" xyz="0 0 0"/>
     <geometry>
-      <cylinder length="0.05" radius="0.12"/>
+      <cylinder length="0.05" radius="0.1"/>
     </geometry>
   </visual>
@@ -83,5 +83,5 @@
     <origin rpy="1.5707963267948966 0 0" xyz="0 0 0"/>
     <geometry>
-      <cylinder length="0.05" radius="0.12"/>
+      <cylinder length="0.05" radius="0.1"/>
     </geometry>
   </collision>
@@ -115,5 +115,5 @@
     <origin rpy="1.5707963267948966 0 0" xyz="0 0 0"/>
     <geometry>
-      <cylinder length="0.05" radius="0.12"/>
+      <cylinder length="0.05" radius="0.1"/>
     </geometry>
   </visual>
@@ -121,9 +121,10 @@
     <origin rpy="1.5707963267948966 0 0" xyz="0 0 0"/>
     <geometry>
-      <cylinder length="0.05" radius="0.12"/>
+      <cylinder length="0.05" radius="0.1"/>
     </geometry>
   </collision>
   </link>
-<link name="camera_link">
+<!-- front_camera -->
+<link name="front_camera_link">
     <collision>
       <origin xyz="0 0 0" rpy="0 0 0"/>
@@ -145,10 +146,90 @@
     </inertial>
   </link>
-  <joint name="camera_joint" type="fixed">
+  <joint name="front_camera_joint" type="fixed">
     <axis xyz="0 1 0" />
-    <origin xyz="0.4 0.0 0.2" rpy="0 0 0"/>
-    <parent link="base_link"/>
-    <child link="camera_link"/>
-  </joint>
+    <origin xyz="0.03 0.0 -0.05" rpy="0 0 0"/>
+    <parent link="front_hokuyo_link"/>
+    <child link="front_camera_link"/>
+  </joint>
+<!-- back_camera -->
+<link name="back_camera_link">
+    <collision>
+      <origin xyz="0 0 0" rpy="0 0 0"/>
+      <geometry>
+    <box size="0.01 0.01 0.01"/>
+      </geometry>
+    </collision>
+    <visual>
+      <origin xyz="0 0 0" rpy="0 0 0"/>
+      <geometry>
+    <box size="0.01 0.01 0.01"/>
+      </geometry>
+      <material name="red"/>
+    </visual>
+    <inertial>
+      <mass value="1e-5" />
+      <origin xyz="0 0 0" rpy="0 0 0"/>
+      <inertia ixx="1e-6" ixy="0" ixz="0" iyy="1e-6" iyz="0" izz="1e-6" />
+    </inertial>
+  </link>
+  <joint name="back_camera_joint" type="fixed">
+    <axis xyz="0 1 0" />
+    <origin xyz="-0.4 0.0 0.15" rpy="0 0 3.1415926"/>
+    <parent link="base_link"/>
+    <child link="back_camera_link"/>
+  </joint>
+  <!-- front Hokuyo Laser -->
+   <joint name="front_hokuyo_joint" type="fixed">
+    <axis xyz="0 1 0" />
+    <origin xyz="0.37 0 0.2" rpy="0 0 0"/>
+    <parent link="base_link"/>
+    <child link="front_hokuyo_link"/>
+  </joint>
+  <link name="front_hokuyo_link">
+    <collision>
+      <origin xyz="0 0 0" rpy="0 0 0"/>
+      <geometry>
+    <box size="0.1 0.1 0.1"/>
+      </geometry>
+    </collision>
+    <visual>
+      <origin xyz="0 0 0" rpy="0 0 0"/>
+      <geometry>
+        <mesh filename="package://convoy_gazebo/urdf/hokuyo.dae"/>
+      </geometry>
+    </visual>
+    <inertial>
+      <mass value="1e-5" />
+      <origin xyz="0 0 0" rpy="0 0 0"/>
+      <inertia ixx="1e-6" ixy="0" ixz="0" iyy="1e-6" iyz="0" izz="1e-6" />
+    </inertial>
+  </link>
+ <!-- back Hokuyo Laser -->
+   <joint name="back_hokuyo_joint" type="fixed">
+    <axis xyz="0 1 0" />
+    <origin xyz="-0.37 0 0.2" rpy="0 0 3.1415926"/>
+    <parent link="base_link"/>
+    <child link="back_hokuyo_link"/>
+  </joint>
+  <link name="back_hokuyo_link">
+    <collision>
+      <origin xyz="0 0 0" rpy="0 0 0"/>
+      <geometry>
+    <box size="0.1 0.1 0.1"/>
+      </geometry>
+    </collision>
+    <visual>
+      <origin xyz="0 0 0" rpy="0 0 0"/>
+      <geometry>
+        <mesh filename="package://convoy_gazebo/urdf/hokuyo.dae"/>
+      </geometry>
+    </visual>
+    <inertial>
+      <mass value="1e-5" />
+      <origin xyz="0 0 0" rpy="0 0 0"/>
+      <inertia ixx="1e-6" ixy="0" ixz="0" iyy="1e-6" iyz="0" izz="1e-6" />
+    </inertial>
+  </link>
+<!--   BLA  -->
   <gazebo reference="right_back_wheel">
     <material>Gazebo/Black</material>
@@ -179,5 +260,5 @@
     <origin rpy="1.5707963267948966 0 0" xyz="0 0 0"/>
     <geometry>
-      <cylinder length="0.05" radius="0.12"/>
+      <cylinder length="0.05" radius="0.1"/>
     </geometry>
   </visual>
@@ -185,5 +266,5 @@
     <origin rpy="1.5707963267948966 0 0" xyz="0 0 0"/>
     <geometry>
-      <cylinder length="0.05" radius="0.12"/>
+      <cylinder length="0.05" radius="0.1"/>
     </geometry>
   </collision>
@@ -225,6 +306,6 @@
 </gazebo>
 <!-- front camera -->
-  <gazebo reference="camera_link">
-    <sensor type="camera" name="camera">
+  <gazebo reference="front_camera_link">
+    <sensor type="camera" name="front_camera">
       <update_rate>30.0</update_rate>
       <camera name="head">
@@ -251,8 +332,8 @@
         <alwaysOn>true</alwaysOn>
         <updateRate>0.0</updateRate>
-        <cameraName>/camera</cameraName>
+        <cameraName>/front_camera</cameraName>
         <imageTopicName>image_raw</imageTopicName>
         <cameraInfoTopicName>camera_info</cameraInfoTopicName>
-        <frameName>camera_link1</frameName>
+        <frameName>front_camera_link</frameName>
         <hackBaseline>0.07</hackBaseline>
         <distortionK1>0.0</distortionK1>
@@ -264,4 +345,117 @@
     </sensor>
   </gazebo>
-  <xacro:property name="camera_link" value="0.05" /> <!-- Size of square 'camera' box -->
+<!-- back camera -->
+  <gazebo reference="back_camera_link">
+    <sensor type="camera" name="back_camera">
+      <update_rate>30.0</update_rate>
+      <camera name="head">
+        <horizontal_fov>2.2</horizontal_fov>
+        <image>
+          <width>640</width>
+          <height>480</height>
+          <format>R8G8B8</format>
+        </image>
+        <clip>
+          <near>0.02</near>
+          <far>300</far>
+        </clip>
+        <noise>
+          <type>gaussian</type>
+          <!-- Noise is sampled independently per pixel on each frame.
+               That pixel's noise value is added to each of its color
+               channels, which at that point lie in the range [0,1]. -->
+          <mean>0.0</mean>
+          <stddev>0.007</stddev>
+        </noise>
+      </camera>
+      <plugin name="camera_controller" filename="libgazebo_ros_camera.so">
+        <alwaysOn>true</alwaysOn>
+        <updateRate>0.0</updateRate>
+        <cameraName>/back_camera</cameraName>
+        <imageTopicName>image_raw</imageTopicName>
+        <cameraInfoTopicName>camera_info</cameraInfoTopicName>
+        <frameName>back_camera_link</frameName>
+        <hackBaseline>0.07</hackBaseline>
+        <distortionK1>0.0</distortionK1>
+        <distortionK2>0.0</distortionK2>
+        <distortionK3>0.0</distortionK3>
+        <distortionT1>0.0</distortionT1>
+        <distortionT2>0.0</distortionT2>
+      </plugin>
+    </sensor>
+  </gazebo>
+   <gazebo reference="front_hokuyo_link">
+    <sensor type="gpu_ray" name="head_hokuyo_sensor">
+      <pose>0 0 0 0 0 0</pose>
+      <visualize>false</visualize>
+      <update_rate>30</update_rate>
+      <ray>
+        <scan>
+          <horizontal>
+            <samples>720</samples>
+            <resolution>1</resolution>
+            <min_angle>-1.570796</min_angle>
+            <max_angle>1.570796</max_angle>
+          </horizontal>
+        </scan>
+        <range>
+          <min>0.10</min>
+          <max>10.0</max>
+          <resolution>0.01</resolution>
+        </range>
+        <noise>
+          <type>gaussian</type>
+          <!-- Noise parameters based on published spec for Hokuyo laser
+               achieving "+-30mm" accuracy at range < 10m.  A mean of 0.0m and
+               stddev of 0.01m will put 99.7% of samples within 0.03m of the true
+               reading. -->
+          <mean>0.0</mean>
+          <stddev>0.01</stddev>
+        </noise>
+      </ray>
+      <plugin name="gazebo_ros_head_hokuyo_controller" filename="libgazebo_ros_gpu_laser.so">
+        <topicName>front_scan</topicName>
+        <frameName>front_hokuyo_link</frameName>
+      </plugin>
+    </sensor>
+  </gazebo>
+   <gazebo reference="back_hokuyo_link">
+    <sensor type="gpu_ray" name="head_hokuyo_sensor">
+      <pose>0 0 0 0 0 0</pose>
+      <visualize>false</visualize>
+      <update_rate>30</update_rate>
+      <ray>
+        <scan>
+          <horizontal>
+            <samples>720</samples>
+            <resolution>1</resolution>
+            <min_angle>-1.570796</min_angle>
+            <max_angle>1.570796</max_angle>
+          </horizontal>
+        </scan>
+        <range>
+          <min>0.10</min>
+          <max>10.0</max>
+          <resolution>0.01</resolution>
+        </range>
+        <noise>
+          <type>gaussian</type>
+          <!-- Noise parameters based on published spec for Hokuyo laser
+               achieving "+-30mm" accuracy at range < 10m.  A mean of 0.0m and
+               stddev of 0.01m will put 99.7% of samples within 0.03m of the true
+               reading. -->
+          <mean>0.0</mean>
+          <stddev>0.01</stddev>
+        </noise>
+      </ray>
+      <plugin name="gazebo_ros_head_hokuyo_controller" filename="libgazebo_ros_gpu_laser.so">
+        <topicName>back_scan</topicName>
+        <frameName>back_hokuyo_link</frameName>
+      </plugin>
+    </sensor>
+  </gazebo>
+  <xacro:property name="front_hokuyo_link" value="0.05" />
+  <xacro:property name="back_hokuyo_link" value="0.05" />
+  <xacro:property name="front_camera_link" value="0.05" />
+  <xacro:property name="back_camera_link" value="0.05" />
 </robot>
