Commit message: Signed-off-by: Or Tslil <ortslil64@gmail.com>

File: urdf/KoBot.urdf.xacro (robot description, xacro)
@@ -204,5 +204,5 @@
       <origin xyz="0 0 0" rpy="0 0 0"/>
       <geometry>
-        <mesh filename="package://SLAM/urdf/hokuyo.dae"/>
+        <mesh filename="package://convoy_gazebo/urdf/hokuyo.dae"/>
       </geometry>
     </visual>

Commit message: Signed-off-by: Or Tslil <ortslil64@gmail.com>

File: urdf/KoBot.urdf.xacro (robot description, xacro)
@@ -49,7 +49,4 @@
   </collision>
   </link>
-  <gazebo reference="right_wheel">
-    <material>Gazebo/Black</material>
-  </gazebo>
   <joint name="base_link_right_wheel" type="continuous">
     <parent link="base_link"/>
@@ -151,7 +148,4 @@
     <child link="camera_link"/>
   </joint>
-  <gazebo reference="right_back_wheel">
-    <material>Gazebo/Black</material>
-  </gazebo>
   <joint name="base_link_right_back_wheel" type="continuous">
     <parent link="base_link"/>
@@ -189,7 +183,4 @@
   </collision>
   </link>
-  <gazebo reference="left_back_wheel">
-    <material>Gazebo/Black</material>
-  </gazebo>
   <joint name="base_link_left_back_wheel" type="continuous">
     <parent link="base_link"/>
@@ -208,4 +199,25 @@
     </joint>
   </transmission>
+<!-- gazebo properties -->
+<gazebo reference="right_wheel">
+    <material>Gazebo/Black</material>
+<mu1>0.5</mu1>
+    <mu2>0.5</mu2>
+  </gazebo>
+<gazebo reference="left_back_wheel">
+    <material>Gazebo/Black</material>
+<mu1>0.8</mu1>
+    <mu2>0.8</mu2>
+  </gazebo>
+<gazebo reference="left_wheel">
+    <material>Gazebo/Black</material>
+<mu1>0.5</mu1>
+    <mu2>0.5</mu2>
+  </gazebo>
+<gazebo reference="right_back_wheel">
+    <material>Gazebo/Black</material>
+    <mu1>0.8</mu1>
+    <mu2>0.8</mu2>
+  </gazebo>
 <gazebo>
     <plugin name="skid_steer_drive_controller" filename="libgazebo_ros_skid_steer_drive.so">
@@ -217,6 +229,6 @@
         <rightRearJoint>base_link_right_back_wheel</rightRearJoint>
         <wheelSeparation>0.545</wheelSeparation>
-        <wheelDiameter>0.2</wheelDiameter>
-        <torque>20</torque>
+        <wheelDiameter>0.24</wheelDiameter>
+        <torque>30</torque>
         <commandTopic>cmd_vel</commandTopic>
         <robotBaseFrame>base_link</robotBaseFrame>

File: urdf/KoBot_ai.urdf.xacro (robot description, xacro)
@@ -49,7 +49,4 @@
   </collision>
   </link>
-  <gazebo reference="right_wheel">
-    <material>Gazebo/Black</material>
-  </gazebo>
   <joint name="base_link_right_wheel" type="continuous">
     <parent link="base_link"/>
@@ -87,7 +84,4 @@
   </collision>
   </link>
-  <gazebo reference="left_wheel">
-    <material>Gazebo/Black</material>
-  </gazebo>
   <joint name="base_link_left_wheel" type="continuous">
     <parent link="base_link"/>
@@ -232,7 +226,4 @@
   </link>
 <!--   BLA  -->
-  <gazebo reference="right_back_wheel">
-    <material>Gazebo/Black</material>
-  </gazebo>
   <joint name="base_link_right_back_wheel" type="continuous">
     <parent link="base_link"/>
@@ -270,7 +261,4 @@
   </collision>
   </link>
-  <gazebo reference="left_back_wheel">
-    <material>Gazebo/Black</material>
-  </gazebo>
   <joint name="base_link_left_back_wheel" type="continuous">
     <parent link="base_link"/>
@@ -299,5 +287,5 @@
         <wheelSeparation>0.545</wheelSeparation>
         <wheelDiameter>0.2</wheelDiameter>
-        <torque>20</torque>
+        <torque>30</torque>
         <commandTopic>cmd_vel</commandTopic>
         <robotBaseFrame>base_link</robotBaseFrame>
@@ -455,4 +443,25 @@
     </sensor>
   </gazebo>
+<!-- gazebo properties -->
+<gazebo reference="right_wheel">
+    <material>Gazebo/Black</material>
+<mu1>0.5</mu1>
+    <mu2>0.5</mu2>
+  </gazebo>
+<gazebo reference="left_back_wheel">
+    <material>Gazebo/Black</material>
+<mu1>0.8</mu1>
+    <mu2>0.8</mu2>
+  </gazebo>
+<gazebo reference="left_wheel">
+    <material>Gazebo/Black</material>
+<mu1>0.5</mu1>
+    <mu2>0.5</mu2>
+  </gazebo>
+<gazebo reference="right_back_wheel">
+    <material>Gazebo/Black</material>
+    <mu1>0.8</mu1>
+    <mu2>0.8</mu2>
+  </gazebo>
   <xacro:property name="front_hokuyo_link" value="0.05" />
   <xacro:property name="back_hokuyo_link" value="0.05" />
